Commit message: updated xacro definitions, shadow hand not integrated, need to check that!

File: clopema_testbed/clopema_description/robots/clopema_LOCAL.urdf.xacro (robot description, xacro)
@@ -1 +1,86 @@
-clopema_UG.urdf.xacro
+<?xml version="1.0"?>
+<robot xmlns:xacro="http://www.ros.org/wiki/xacro" name="clopema">
+	<xacro:include filename="$(find clopema_description)/urdf/common.urdf.xacro" />
+	<xacro:include filename="$(find clopema_description)/urdf/room_ug.urdf.xacro" />
+	<xacro:include filename="$(find clopema_description)/urdf/base_link.urdf.xacro" />
+	<xacro:include filename="$(find clopema_description)/urdf/ma1400/ma1400.urdf.xacro" />
+	<xacro:include filename="$(find clopema_description)/urdf/gripper.urdf.xacro" />
+	<xacro:include filename="$(find clopema_description)/urdf/r750.urdf.xacro" />
+<!--	<xacro:include filename="$(find clopema_description)/urdf/table.urdf.xacro" />	-->
+	<xacro:include filename="$(find clopema_description)/urdf/table_adjustable.urdf.xacro" />
+	<xacro:include filename="$(find clopema_description)/urdf/colObjects.urdf.xacro" />
+	<xacro:include filename="$(find clopema_description)/urdf/xtion.urdf.xacro" />
+	<xacro:include filename="$(find clopema_description)/urdf/alvar_marker_UG.urdf.xacro" />
+	<xacro:include filename="$(find clopema_description)/urdf/robot_head_UG.xacro" />
+	<xacro:base_link/>
+	<xacro:room_ug/>
+	<xacro:r750 parent="base_link" suffix="" color="blue">
+		<origin xyz="0.0 0.0 0.011" rpy="0 0 0"/>
+	</xacro:r750>
+	<xacro:ma1400 parent="r750" suffix="r1_" color="blue">
+		<origin xyz="0 -.25 0.1600" rpy="${15*TO_RAD} 0 0"/>
+	</xacro:ma1400>
+	<xacro:ma1400 parent="r750" suffix="r2_" color="blue">
+		<origin xyz="0 .25 0.1600" rpy="-${15*TO_RAD} 0 0"/>
+	</xacro:ma1400>
+	<xacro:gripper parent="tip_link" suffix="r1_" color="blue">
+		<origin xyz="0.000 0 0.02" rpy="0 0 ${PI/2+PI/6}"/>
+	</xacro:gripper>
+	<xacro:gripper parent="tip_link" suffix="r2_" color="blue">
+		<origin xyz="0.000 0 0.02" rpy="0 0 ${PI/2+PI/6}"/>
+	</xacro:gripper>
+	<link name="torso_link"/>
+	<joint name="torso_link_f" type="fixed">
+		  <child link="torso_link"/>
+		  <parent link="r750"/>
+		  <origin xyz="0 0 -0.51" rpy="0 0 ${PI/2}"/>
+	</joint>
+<!--	<xacro:robot_head parent="torso_link" b_roll="-7.57715255e-02" b_pitch="-2.22676038e-03" b_yaw="9.94329993e-03" b_x="-3.02628815e-01" b_y="3.17237899e-02" b_z="2.15836964e-03">-->
+<!--		<origin rpy="${45*TO_RAD} 0 0" xyz="1.6529e-06 0.45 2.31511"/>-->
+<!--    </xacro:robot_head>-->
+    <xacro:robot_head parent="r750">
+        <origin rpy="0 0 0" xyz="-0.45 0.15 1.68"/>
+    </xacro:robot_head>
+	<xacro:alvar_marker parent="r1_tip_link" prefix="r1" width="0.052" offset="-0.0322">
+        <origin xyz="0 0 0.06288" rpy="0 0 -${60*TO_RAD}"/>
+    </xacro:alvar_marker>
+    <link name="calib_target"> </link>
+    <joint name="calib_target_joint" type="fixed">
+        <origin xyz="0 -0.92 0.70" rpy="0 0 0"/>
+        <parent link="base_link"/>
+        <child link="calib_target"/>
+    </joint>
+	<xacro:colObjects/>
+	<xacro:xtion parent="r2_link_6" suffix="2" prefix="" color="grey">
+        <origin xyz="-0.13 -0.15 0" rpy="0 ${-PI/2} 0"/>
+    </xacro:xtion>
+    <xacro:xtion parent="r1_link_6" suffix="1" prefix="" color="grey">
+        <origin xyz="-0.13 -0.15 0" rpy="0 ${-PI/2} 0"/>
+    </xacro:xtion>
+    <xacro:xtion parent="torso_link" suffix="3" prefix="" color="grey">
+        <origin xyz="0 0 -50.0" rpy="0 0 0"/> <!-- Go away if not calibrated -->
+    </xacro:xtion>
+	<xacro:table parent="base_link" suffix="t1_" color="grey" height="0.70" deskx="0.8" desky="0.8">
+		<origin xyz="1.0 0.0 0.70" rpy="0 0 0"/>
+	</xacro:table>
+	<xacro:table parent="base_link" suffix="t2_" color="grey" height="0.70" deskx="0.8" desky="0.8">
+		<origin xyz="0.0 -1.2 0.70" rpy="0 0 0"/>
+	</xacro:table>
+	<!--Markers on the table for flattening-->
+<!--	<xacro:alvar_marker parent="t2_leg_2" suffix="t2_tL" width="0.06">-->
+<!--        <origin xyz="0.035 0.035 0" rpy="0 0 ${90*TO_RAD}"/>-->
+<!--    </xacro:alvar_marker>-->
+<!--    <xacro:alvar_marker parent="t2_leg_3" suffix="t2_tR" width="0.06">-->
+<!--        <origin xyz="0.035 0.035 0" rpy="0 0 ${180*TO_RAD}"/>-->
+<!--    </xacro:alvar_marker>-->
+<!--    <xacro:alvar_marker parent="t2_leg_1" suffix="t2_bL" width="0.06">-->
+<!--        <origin xyz="0.035 0.035 0" rpy="0 0 0"/>-->
+<!--    </xacro:alvar_marker>-->
+<!--    <xacro:alvar_marker parent="t2_leg_4" suffix="t2_bR" width="0.06">-->
+<!--        <origin xyz="0.035 0.035 0" rpy="0 0 -${90*TO_RAD}"/>-->
+<!--    </xacro:alvar_marker>-->
+    <!--Markers on the table for flattening-->
+	<xacro:table parent="base_link" suffix="t3_" color="grey" height="0.70" deskx="0.8" desky="0.8">
+		<origin xyz="-1.0 0.0 0.70" rpy="0 0 0"/>
+	</xacro:table>
+</robot>

File: clopema_testbed/clopema_description/urdf/alvar_marker.urdf.xacro (robot description, xacro)
@@ -8,5 +8,5 @@
 		<link name="alvar_${suffix}_rightUp"></link>
 		<joint name="alvar_${suffix}_center_joint" type="fixed">
-			<insert_block name="origin"/>
+			<xacro:insert_block name="origin"/>
 			<parent link="${parent}"/>
 			<child link="alvar_${suffix}_center" />

File: clopema_testbed/clopema_description/urdf/alvar_marker_UG.urdf.xacro (robot description, xacro)
@@ -9,5 +9,5 @@
 		<link name="alvar_${prefix}_rightUp"></link>
 		<joint name="alvar_${prefix}_corrOrient_joint" type="fixed">
-			<insert_block name="origin"/>
+			<xacro:insert_block name="origin"/>
 			<parent link="${parent}"/>
 			<child link="alvar_${prefix}_corrOrient" />

File: clopema_testbed/clopema_description/urdf/colObjects.urdf.xacro (robot description, xacro)
@@ -11,5 +11,5 @@
 		</link>
 		<joint name="${suffix}joint_f_cable_1" type="fixed">
-			<insert_block name="origin" />
+			<xacro:insert_block name="origin" />
 			<parent link="${parent}"/>
 			<child link="${suffix}cable_1"/>
@@ -36,10 +36,10 @@
 		</link>
 		<joint name="${prefix}joint_fkinect${suffix}" type="fixed">
-			<insert_block name="origin" />
+			<xacro:insert_block name="origin" />
 			<parent link="${parent}"/>
 			<child link="${prefix}xtion${suffix}"/>
 		</joint>
 		<joint name="${prefix}joint_fkinect${suffix}_ee" type="fixed">
-			<insert_block name="origin" />
+			<xacro:insert_block name="origin" />
 			<parent link="${parent}"/>
 			<child link="${prefix}xtion${suffix}_ee"/>
@@ -80,5 +80,5 @@
 		</link>
 		<joint name="${suffix}joint_fcamera_stick" type="fixed">
-			<insert_block name="origin" />
+			<xacro:insert_block name="origin" />
 			<parent link="${parent}"/>
 			<child link="${suffix}camera_stick"/>

File: clopema_testbed/clopema_description/urdf/d46.urdf.xacro (robot description, xacro)
@@ -1,5 +1,4 @@
 <?xml version="1.0"?>
-<robot name="ptu_d46"
-       xmlns:xacro="http://ros.org/wiki/xacro">
+<robot xmlns:xacro="http://www.ros.org/wiki/xacro">
   <xacro:property name="pan_velocity" value="1.0" />
   <xacro:property name="pan_range" value="2.775" />

File: clopema_testbed/clopema_description/urdf/dx100.urdf.xacro (robot description, xacro)
@@ -19,5 +19,5 @@
 		</link>
 		<joint name="joint_f_dx100" type="fixed">
-			<insert_block name="origin" />
+			<xacro:insert_block name="origin" />
 			<parent link="${parent}"/>
 			<child link="dx100"/>

File: clopema_testbed/clopema_description/urdf/force_sensor.urdf.xacro (robot description, xacro)
@@ -13,5 +13,5 @@
        </link>
        <joint name="${suffix}force_sensor_joint_f" type="fixed">
-           <insert_block name="origin" />
+           <xacro:insert_block name="origin" />
            <parent link="${suffix}${parent}"/>
            <child link="${suffix}force_sensor"/>

File: clopema_testbed/clopema_description/urdf/gripper.urdf.xacro (robot description, xacro)
@@ -20,5 +20,5 @@
 		<joint name="${suffix}joint_fgrip" type="fixed">
 			<child link="${suffix}gripper"/>
-			<insert_block name="origin" />
+			<xacro:insert_block name="origin" />
 			<parent link="${suffix}${parent}"/>
 		</joint>
@@ -40,5 +40,5 @@
 			<limit lower="0" upper="1" velocity="1000.0" effort="1000.0" />
 			<child link="${suffix}gripper_status"/>
-			<insert_block name="origin" />
+			<xacro:insert_block name="origin" />
 			<parent link="${suffix}gripper"/>
 		</joint>

File: clopema_testbed/clopema_description/urdf/gripper_v2.urdf.xacro (robot description, xacro)
@@ -20,5 +20,5 @@
 		<joint name="${suffix}joint_fgrip" type="fixed">
 			<child link="${suffix}gripper"/>
-			<insert_block name="origin" />
+			<xacro:insert_block name="origin" />
 			<parent link="${suffix}${parent}"/>
 		</joint>
@@ -46,5 +46,5 @@
 			<limit lower="0" upper="1" velocity="1000.0" effort="1000.0" />
 			<child link="${suffix}gripper_status"/>
-			<insert_block name="origin" />
+			<xacro:insert_block name="origin" />
 			<parent link="${suffix}gripper"/>
 		</joint>

File: clopema_testbed/clopema_description/urdf/gripper_v3.urdf.xacro (robot description, xacro)
@@ -24,5 +24,5 @@
                 <joint name="${suffix}joint_fgrip" type="fixed">
                         <child link="${suffix}gripper"/>
-                        <insert_block name="origin" />
+                        <xacro:insert_block name="origin" />
                         <parent link="${suffix}${parent}"/>
                 </joint>
@@ -50,5 +50,5 @@
                         <limit lower="0" upper="1" velocity="1000.0" effort="1000.0" />
                         <child link="${suffix}gripper_status"/>
-                        <insert_block name="origin" />
+                        <xacro:insert_block name="origin" />
                         <parent link="${suffix}gripper"/>
                 </joint>

File: clopema_testbed/clopema_description/urdf/hanging_string.xacro (robot description, xacro)
@@ -24,5 +24,5 @@
         </link>
         <joint name="joint_stand_${suffix}" type="fixed">
-            <insert_block name="origin" />
+            <xacro:insert_block name="origin" />
             <parent link="${parent}"/>
             <child link="stand_${suffix}"/>
@@ -34,5 +34,5 @@
         <link name="hanging_string_floor_center" />
         <joint name="joint_hanging_string_floor_center" type="fixed">
-            <insert_block name="origin" />
+            <xacro:insert_block name="origin" />
             <parent link="${parent}"/>
             <child link="hanging_string_floor_center"/>

File: clopema_testbed/clopema_description/urdf/ma1400/link_1.urdf.xacro (robot description, xacro)
@@ -19,5 +19,5 @@
 		</link>
 		<joint name="${suffix}joint_f1" type="fixed">
-			<insert_block name="origin" />
+			<xacro:insert_block name="origin" />
 			<parent link="${parent}"/>
 			<child link="${suffix}link_1"/>

File: clopema_testbed/clopema_description/urdf/ma1400/link_2.urdf.xacro (robot description, xacro)
@@ -22,5 +22,5 @@
 			<limit lower="-${170*TO_RAD}" upper="${170*TO_RAD}" velocity="${220*TO_RAD}" effort="1000.0" />
 			<child link="${suffix}link_2"/>
-			<insert_block name="origin" />
+			<xacro:insert_block name="origin" />
 			<parent link="${suffix}${parent}"/>
 		</joint>

File: clopema_testbed/clopema_description/urdf/ma1400/link_3.urdf.xacro (robot description, xacro)
@@ -22,5 +22,5 @@
 			<limit lower="-${90*TO_RAD}" upper="${155*TO_RAD}" velocity="${200*TO_RAD}" effort="1000.0" />
 			<child link="${suffix}link_3"/>
-			<insert_block name="origin" />
+			<xacro:insert_block name="origin" />
 			<parent link="${suffix}${parent}"/>
 		</joint>

File: clopema_testbed/clopema_description/urdf/ma1400/link_4.urdf.xacro (robot description, xacro)
@@ -22,5 +22,5 @@
 			<limit lower="-${80*TO_RAD}" upper="${92*TO_RAD}" velocity="${220*TO_RAD}" effort="1000.0" />
 			<child link="${suffix}link_4"/>
-			<insert_block name="origin" />
+			<xacro:insert_block name="origin" />
 			<parent link="${suffix}${parent}"/>
 		</joint>

File: clopema_testbed/clopema_description/urdf/ma1400/link_5.urdf.xacro (robot description, xacro)
@@ -22,5 +22,5 @@
 			<limit lower="-${150*TO_RAD}" upper="${150*TO_RAD}" velocity="${410*TO_RAD}" effort="1000.0" />
 			<child link="${suffix}link_5"/>
-			<insert_block name="origin" />
+			<xacro:insert_block name="origin" />
 			<parent link="${suffix}${parent}"/>
 		</joint>

File: clopema_testbed/clopema_description/urdf/ma1400/link_6.urdf.xacro (robot description, xacro)
@@ -22,5 +22,5 @@
 			<limit lower="-${45*TO_RAD}" upper="${180*TO_RAD}" velocity="${410*TO_RAD}" effort="1000.0" />
 			<child link="${suffix}link_6"/>
-			<insert_block name="origin" />
+			<xacro:insert_block name="origin" />
 			<parent link="${suffix}${parent}"/>
 		</joint>

File: clopema_testbed/clopema_description/urdf/ma1400/ma1400.urdf.xacro (robot description, xacro)
@@ -10,5 +10,5 @@
 	<xacro:macro name="ma1400" params="*origin parent suffix color">
 		<xacro:link_1 parent="${parent}" suffix="${suffix}" color="${color}">
-			<insert_block name="origin" />
+			<xacro:insert_block name="origin" />
 		</xacro:link_1>
 		<xacro:link_2 parent="link_1" suffix="${suffix}" color="${color}">

File: clopema_testbed/clopema_description/urdf/ma1400/tip_link.urdf.xacro (robot description, xacro)
@@ -12,5 +12,5 @@
 			<limit lower="-${199*TO_RAD}" upper="${199*TO_RAD}" velocity="${610*TO_RAD}" effort="1000.0" />
 			<child link="${suffix}link_7"/>
-			<insert_block name="origin" />
+			<xacro:insert_block name="origin" />
 			<parent link="${suffix}${parent}"/>
 		</joint>

File: clopema_testbed/clopema_description/urdf/r750.urdf.xacro (robot description, xacro)
@@ -42,5 +42,5 @@
 		</joint>
 		<joint name="${suffix}joint_f0" type="fixed">
-			<insert_block name="origin" />
+			<xacro:insert_block name="origin" />
 			<parent link="${parent}"/>
 			<child link="${suffix}r750_base"/>
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